Commit message: Fix path to stl files

File: models/mevius.urdf (robot description, URDF)
Before this commit: robot mevius, 17 links, 16 joints
Links:
- link BL_calf_link: geometry collision cylinder length=0.23 radius=0.01; visual mesh filename=./meshes/BL_calf_link.STL
- link BL_scapula_link: geometry collision cylinder length=0.08 radius=0.05; visual mesh filename=./meshes/BL_scapula_link.STL
- link BL_thigh_link: geometry visual mesh filename=./meshes/BL_thigh_link.STL
- link BR_calf_link: geometry collision cylinder length=0.23 radius=0.01; visual mesh filename=./meshes/BR_calf_link.STL
- link BR_scapula_link: geometry collision cylinder length=0.08 radius=0.05; visual mesh filename=./meshes/BR_scapula_link.STL
- link BR_thigh_link: geometry visual mesh filename=./meshes/BR_thigh_link.STL
- link FL_calf_link: geometry collision cylinder length=0.23 radius=0.01; visual mesh filename=./meshes/FL_calf_link.STL
- link FL_scapula_link: geometry collision cylinder length=0.08 radius=0.05; visual mesh filename=./meshes/FL_scapula_link.STL
- link FL_thigh_link: geometry visual mesh filename=./meshes/FL_thigh_link.STL
- link FR_calf_link: geometry collision cylinder length=0.23 radius=0.01; visual mesh filename=./meshes/FR_calf_link.STL
- link FR_scapula_link: geometry collision cylinder length=0.08 radius=0.05; visual mesh filename=./meshes/FR_scapula_link.STL
- link FR_thigh_link: geometry visual mesh filename=./meshes/FR_thigh_link.STL
- link base_link: geometry collision box size=0.334 0.200 0.150; visual mesh filename=meshes/base_link.STL
